Commit message: sdsd

File: rob_ws/src/wheelchair_bringup/urdf/wheelchair.urdf (robot description, URDF)
Before this commit: robot wheelchair, 2 links, 1 joints
Links:
- added link ultrasonic_link; visual box size=0.04 0.04 0.02
Joints:
- added joint ultrasonic_joint: type fixed, parent base_link, child ultrasonic_link, origin xyz=0.56 0.27 0.00 rpy=0.0 0.0 0.0
- joint camera_joint: origin xyz=0.22 0.0 1.07 rpy=0 0 0 -> xyz=0.00 -0.23 1.09 rpy=0 0 0
